File: reloj/reloj_smd.kicad_sch (KiCad schematic)
At the start: 15 parts, among them J1 Barrel_Jack, J2 Barrel_Jack, J3 Conn_01x02, U1 NE555P

Commit message: agregar borradores
Parts:
- removed U1: NE555P, Package_DIP:DIP-8_W7.62mm_Socket_LongPads, symbol Timer:NE555P
- added U1: NE555D, Package_SO:SOIC-8_3.9x4.9mm_P1.27mm, symbol Timer:NE555D
Connections:
- net GND: now also U1.1 (GND)
- net VDC: now also U1.4 (~{RST}), U1.8 (VCC)
- net at R1.2, RV1.2: now also U1.7 (DISCH)
- net at C1.1, RV1.3: now also U1.2 (TRIG), U1.6 (THRES)
- net at C2.1: now also U1.5 (CONT)
- net at D1.2 (A), J3.1 (Pin_1): now also U1.3 (OUT)
Changed lines of the file:
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@@
 		)
 		(instances
-			(project "reloj"
+			(project "reloj_smd"
 				(path "/fe13e28c-ea94-4bcc-9b18-67f88f1c47ae"
 					(reference "RV1")
@@
 		)
 		(instances
-			(project "reloj"
+			(project "reloj_smd"
 				(path "/fe13e28c-ea94-4bcc-9b18-67f88f1c47ae"
 					(reference "#PWR010")
+					(unit 1)
+				)
+			)
+		)
+	)
+	(symbol
+		(lib_id "Timer:NE555D")
+		(at 99.06 109.22 0)
+		(unit 1)
+		(body_style 1)
+		(exclude_from_sim no)
+		(in_bom yes)
+		(on_board yes)
+		(in_pos_files yes)
+		(dnp no)
+		(fields_autoplaced yes)
+		(property "Reference" "U1"
+			(at 111.76 102.7998 0)
+			(show_name no)
+			(do_not_autoplace no)
+			(effects
+				(font
+					(size 1.27 1.27)
+				)
+			)
+		)
+		(property "Value" "NE555D"
+			(at 111.76 105.3398 0)
+			(show_name no)
+			(do_not_autoplace no)
+			(effects
+				(font
+					(size 1.27 1.27)
+				)
+			)
+		)
+		(property "Footprint" "Package_SO:SOIC-8_3.9x4.9mm_P1.27mm"
+			(at 99.06 133.35 0)
+			(hide yes)
+			(show_name no)
+			(do_not_autoplace no)
+			(effects
+				(font
+					(size 1.27 1.27)
+				)
+			)
+		)
+		(property "Datasheet" "http://www.ti.com/lit/ds/symlink/ne555.pdf"
+			(at 99.06 135.89 0)
+			(hide yes)
+			(show_name no)
+			(do_not_autoplace no)
+			(effects
+				(font
+					(size 1.27 1.27)
+				)
+			)
+		)
+		(property "Description" "Precision Timers, 555 compatible, SOIC-8"
+			(at 99.06 130.81 0)
+			(hide yes)
+			(show_name no)
+			(do_not_autoplace no)
+			(effects
+				(font
+					(size 1.27 1.27)
+				)
+			)
+		)
+		(pin "1"
+		)
+		(pin "8"
+		)
+		(pin "2"
+		)
+		(pin "3"
+		)
+		(pin "4"
+		)
+		(pin "5"
+		)
+		(pin "6"
+		)
+		(pin "7"
+		)
+		(instances
+			(project "reloj_smd"
+				(path "/fe13e28c-ea94-4bcc-9b18-67f88f1c47ae"
+					(reference "U1")
 					(unit 1)
 				)
@@
 		)
 		(instances
-			(project "reloj"
+			(project "reloj_smd"
 				(path "/fe13e28c-ea94-4bcc-9b18-67f88f1c47ae"
 					(reference "#PWR012")
@@
 		)
 		(instances
-			(project "reloj"
+			(project "reloj_smd"
 				(path "/fe13e28c-ea94-4bcc-9b18-67f88f1c47ae"
 					(reference "C2")
-					(unit 1)
-				)
-			)
-		)
-	)
-	(symbol
-		(lib_id "Timer:NE555P")
-		(at 99.06 109.22 0)
-		(unit 1)
-		(body_style 1)
-		(exclude_from_sim no)
-		(in_bom yes)
-		(on_board yes)
-		(in_pos_files yes)
-		(dnp no)
-		(fields_autoplaced yes)
-		(property "Reference" "U1"
-			(at 111.76 102.7998 0)
-			(show_name no)
-			(do_not_autoplace no)
-			(effects
-				(font
-					(size 1.27 1.27)
-				)
-			)
-		)
-		(property "Value" "NE555P"
-			(at 111.76 105.3398 0)
-			(show_name no)
-			(do_not_autoplace no)
-			(effects
-				(font
-					(size 1.27 1.27)
-				)
-			)
-		)
-		(property "Footprint" "Package_DIP:DIP-8_W7.62mm_Socket_LongPads"
-			(at 99.06 133.35 0)
-			(hide yes)
-			(show_name no)
-			(do_not_autoplace no)
-			(effects
-				(font
-					(size 1.27 1.27)
-				)
-			)
-		)
-		(property "Datasheet" "http://www.ti.com/lit/ds/symlink/ne555.pdf"
-			(at 99.06 135.89 0)
-			(hide yes)
-			(show_name no)
-			(do_not_autoplace no)
-			(effects
-				(font
-					(size 1.27 1.27)
-				)
-			)
-		)
-		(property "Description" "Precision Timers, 555 compatible, PDIP-8"
-			(at 99.06 130.81 0)
-			(hide yes)
-			(show_name no)
-			(do_not_autoplace no)
-			(effects
-				(font
-					(size 1.27 1.27)
-				)
-			)
-		)
-		(pin "2"
-		)
-		(pin "8"
-		)
-		(pin "1"
-		)
-		(pin "4"
-		)
-		(pin "5"
-		)
-		(pin "3"
-		)
-		(pin "6"
-		)
-		(pin "7"
-		)
-		(instances
-			(project "reloj"
-				(path "/fe13e28c-ea94-4bcc-9b18-67f88f1c47ae"
-					(reference "U1")
 					(unit 1)
 				)
@@
 		)
 		(instances
-			(project "reloj"
+			(project "reloj_smd"
 				(path "/fe13e28c-ea94-4bcc-9b18-67f88f1c47ae"
 					(reference "D1")
@@
 		)
 		(instances
-			(project "reloj"
+			(project "reloj_smd"
 				(path "/fe13e28c-ea94-4bcc-9b18-67f88f1c47ae"
 					(reference "R3")
@@
 		)
 		(instances
-			(project "reloj"
+			(project "reloj_smd"
 				(path "/fe13e28c-ea94-4bcc-9b18-67f88f1c47ae"
 					(reference "#PWR08")
@@
 		)
 		(instances
-			(project "reloj"
+			(project "reloj_smd"
 				(path "/fe13e28c-ea94-4bcc-9b18-67f88f1c47ae"
 					(reference "#PWR09")
@@
 		)
 		(instances
-			(project "reloj"
+			(project "reloj_smd"
 				(path "/fe13e28c-ea94-4bcc-9b18-67f88f1c47ae"
 					(reference "#PWR04")
@@
 		)
 		(instances
-			(project "reloj"
+			(project "reloj_smd"
 				(path "/fe13e28c-ea94-4bcc-9b18-67f88f1c47ae"
 					(reference "#PWR01")
@@
 		)
 		(instances
-			(project "reloj"
+			(project "reloj_smd"
 				(path "/fe13e28c-ea94-4bcc-9b18-67f88f1c47ae"
 					(reference "J1")
@@
 		)
 		(instances
-			(project "reloj"
+			(project "reloj_smd"
 				(path "/fe13e28c-ea94-4bcc-9b18-67f88f1c47ae"
 					(reference "#PWR03")
@@
 		)
 		(instances
-			(project "reloj"
+			(project "reloj_smd"
 				(path "/fe13e28c-ea94-4bcc-9b18-67f88f1c47ae"
 					(reference "C1")
@@
 		)
 		(instances
-			(project "reloj"
+			(project "reloj_smd"
 				(path "/fe13e28c-ea94-4bcc-9b18-67f88f1c47ae"
 					(reference "C3")
@@
 		)
 		(instances
-			(project "reloj"
+			(project "reloj_smd"
 				(path "/fe13e28c-ea94-4bcc-9b18-67f88f1c47ae"
 					(reference "#PWR05")
@@
 		)
 		(instances
-			(project "reloj"
+			(project "reloj_smd"
 				(path "/fe13e28c-ea94-4bcc-9b18-67f88f1c47ae"
 					(reference "D3")
@@
 		)
 		(instances
-			(project "reloj"
+			(project "reloj_smd"
 				(path "/fe13e28c-ea94-4bcc-9b18-67f88f1c47ae"
 					(reference "R2")
@@
 		)
 		(instances
-			(project "reloj"
+			(project "reloj_smd"
 				(path "/fe13e28c-ea94-4bcc-9b18-67f88f1c47ae"
 					(reference "J3")
@@
 		)
 		(instances
-			(project "reloj"
+			(project "reloj_smd"
 				(path "/fe13e28c-ea94-4bcc-9b18-67f88f1c47ae"
 					(reference "#PWR07")
@@
 		)
 		(instances
-			(project "reloj"
+			(project "reloj_smd"
 				(path "/fe13e28c-ea94-4bcc-9b18-67f88f1c47ae"
 					(reference "J2")
@@
 		)
 		(instances
-			(project "reloj"
+			(project "reloj_smd"
 				(path "/fe13e28c-ea94-4bcc-9b18-67f88f1c47ae"
 					(reference "R1")
@@
 		)
 		(instances
-			(project "reloj"
+			(project "reloj_smd"
 				(path "/fe13e28c-ea94-4bcc-9b18-67f88f1c47ae"
 					(reference "#PWR06")
@@
 		)
 		(instances
-			(project "reloj"
+			(project "reloj_smd"
 				(path "/fe13e28c-ea94-4bcc-9b18-67f88f1c47ae"
 					(reference "#PWR02")
@@
 		)
 		(instances
-			(project "reloj"
+			(project "reloj_smd"
 				(path "/fe13e28c-ea94-4bcc-9b18-67f88f1c47ae"
 					(reference "C4")
@@
 		)
 		(instances
-			(project "reloj"
+			(project "reloj_smd"
 				(path "/fe13e28c-ea94-4bcc-9b18-67f88f1c47ae"
 					(reference "#PWR011")
@@
 		)
 		(instances
-			(project "reloj"
+			(project "reloj_smd"
 				(path "/fe13e28c-ea94-4bcc-9b18-67f88f1c47ae"
 					(reference "D2")
